Commit message: Fix joint6 limits and update MoveIt configuration

File: src/my_robot_description/urdf/arm.xacro (robot description, xacro)
@@ -147,4 +147,5 @@
         <origin xyz="0 0 0.05" rpy="0 0 0" />
         <axis xyz="0 0 1" />
+        <limit effort="1000.0" velocity="1.0"/>
     </joint>
     <joint name="hand_tool_joint" type="fixed">
